Commit message: Add lidar

File: description/gazebo_control.xacro (robot description, xacro)
@@ -13,5 +13,5 @@
         <right_joint>right_rear_wheel_joint</right_joint>
         <!-- kinematics -->
-        <wheel_separation>${chassis_width+(wheel_width/2)}</wheel_separation>
+        <wheel_separation>${chassis_width+wheel_width}</wheel_separation>
         <wheel_diameter>${2*wheel_radius}</wheel_diameter>
         <!-- limits -->

File: description/robot.urdf.xacro (robot description, xacro)
@@ -3,3 +3,4 @@
     <xacro:include filename="robot_core.xacro" />
     <xacro:include filename="gazebo_control.xacro"/>
+    <xacro:include filename="lidar.xacro"/>
 </robot>

File: description/robot_core.xacro (robot description, xacro)
@@ -15,4 +15,7 @@
     <material name="black">
         <color rgba="0 0 0 1"/>
+    </material>
+    <material name="green">
+        <color rgba="0 1 0 1"/>
     </material>
     <!--base link-->
